File: hardware/adapter.sch (KiCad schematic (older format))
At the start: 4 parts, among them J1 Conn_02x14_Counter_Clockwise, J2 Conn_01x03_Male, U1 ATtiny814-SS

Commit message: New PCB changes
Other:
- note removed: "FIXME: Pullup R3 on reset line is no longer needed"
- note removed: "FIXME: Short C8 to allow UPDI programming via DTR"
- note removed: "TODO: Check if Pullups on SDA/SCL/INT lines are really enabled"
Changed lines of the file:
@@
 	0    -1   -1   0
 $EndComp
-Text Notes 2300 1150 0    50   ~ 0
-FIXME: Pullup R3 on reset line is no longer needed
-Text Notes 2300 1250 0    50   ~ 0
-FIXME: Short C8 to allow UPDI programming via DTR
 Text GLabel 1900 2500 0    50   Output ~ 0
 TXO
@@
 Text GLabel 3100 3000 2    50   Input ~ 0
 CONFIG
-Text Notes 2300 1350 0    50   ~ 0
-TODO: Check if Pullups on SDA/SCL/INT lines are really enabled
 $Comp
 L power:+3V3 #PWR0105
