File: hardware/sclock_new/sclock_new.sch (KiCad schematic (older format))
At the start: 49 parts, among them J1 Conn_02x03_Odd_Even, J2 Conn_FTDI, J3 Screw_Terminal_01x02, J4 Conn_01x03_Male, J5 Screw_Terminal_01x02, Q1 MMBT3904, Q2 MMBT3904, Q3 MMBT3904, Q4 MMBT3906, Q5 MMBT3904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

Commit message: New PCB changes
Parts:
- added Q7: Si2323CDS, Package_TO_SOT_SMD:SOT-23_Handsoldering, symbol Device:Q_PMOS_GSD
- added R11, R12, R13: 1M, Resistor_SMD:R_0805_2012Metric_Pad1.20x1.40mm_HandSolder, symbol Device:R
- BT1: value c -> 1066
- C4, C7: Value Modifier 35V -> 35V 10%
- C5, C8: footprint Capacitor_SMD:C_0805_2012Metric_Pad1.18x1.45mm_HandSolder -> Capacitor_Tantalum_SMD:CP_EIA-3216-18_Kemet-A_Pad1.58x1.35mm_HandSolder; MPN C0805C106K8PACTU -> T494A106K010AT; Value Modifier 10V X5R -> 10V 10%
- D2, D3, D4, D5: footprint Diode_SMD:D_SOD-323 -> Diode_SMD:D_SOD-323_HandSoldering
- H1, H2, H3, H4: Value Modifier M2 -> M3
- Q1, Q2, Q3, Q4, Q5, Q6: footprint Package_TO_SOT_SMD:SOT-23 -> Package_TO_SOT_SMD:SOT-23_Handsoldering
Connections:
- net GND: now also Q7.1 (G), R11.2, R12.2, R13.2
- net SHDN: now also R13.1
- net VCC: now also Q7.2 (S); no longer SW3.3 (C)
- net at Q2.1 (B), R2.2: now also R12.1
- net at Q1.1 (B), R1.2: now also R11.1
- new net: Q7.3 (D), SW3.3 (C)
Other:
- note added: "M3 Mouting Holes"
- note added: "Reverse Current Protection"
- note removed: "M2 Mouting Holes"
- moved on the sheet: R1, R2, SW3
