File: hardware/sclock_new/sclock_new.kicad_sch (KiCad schematic)
At the start: 53 parts, among them J1 Conn_02x03_Odd_Even, J2 Conn_FTDI, J3 Screw_Terminal_01x02, J4 Conn_01x03_Male, J5 Screw_Terminal_01x02, Q1 MMBT3904, Q2 MMBT3904, Q3 MMBT3904, Q4 MMBT3906, Q5 MMBT3904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

Commit message: PCB v1.1
Parts:
- removed U1: ATtiny814-SS, Package_SO:SOIC-14_3.9x8.7mm_P1.27mm, symbol MCU_Microchip_ATtiny:ATtiny814-SS
- added C9: 0.1µF, Capacitor_SMD:C_0805_2012Metric_Pad1.18x1.45mm_HandSolder, symbol Device:C
- added D10, D7, D8, D9: LED, LED_SMD:LED_0805_2012Metric_Pad1.15x1.40mm_HandSolder, symbol Device:LED
- added R14, R15, R16, R17: 470, Resistor_SMD:R_0805_2012Metric_Pad1.20x1.40mm_HandSolder, symbol Device:R
- added U1: ATtiny816-S, Package_SO:SOIC-20W_7.5x12.8mm_P1.27mm, symbol MCU_Microchip_ATtiny:ATtiny816-S
- C4, C5, C7, C8: symbol Device:CP -> Device:C_Polarized
- D1: MPN 150080YS75000 -> 150080VS75000; Value Modifier 590nm Yellow -> 570nm Green
- Q7: value Si2323CDS -> TSM2323CX; MPN SI2323CDS-T1-GE3 -> TSM2323CX RFG
Connections:
- net +3V3: now also C9.1, U1.1 (VCC)
- net CONFIG: now also U1.17 (PA1)
- net CPULSE1: now also U1.19 (PA3)
- net CPULSE2: now also U1.2 (PA4)
- net GND: now also C9.2, D10.1 (K), D7.1 (K), D8.1 (K), D9.1 (K), U1.20 (GND)
- net INT: now also U1.4 (PA6)
- net LED: now also U1.5 (PA7)
- net RESET: now also U1.18 (PA2)
- net RXI: now also U1.8 (PB3)
- net SCL: now also U1.11 (PB0)
- net SDA: now also U1.10 (PB1)
- net SHDN: now also U1.3 (PA5)
- net TXO: now also U1.9 (PB2)
- net UPDI: now also U1.16 (~{RESET}/PA0)
- new net: D9.2 (A), R16.2
- new net: D10.2 (A), R17.2
- new net: D8.2 (A), R15.2
- new net: D7.2 (A), R14.2
- new net CLED0: R17.1, U1.12 (PC0)
- new net CLED1: R16.1, U1.13 (PC1)
- new net CLED2: R15.1, U1.14 (PC2)
- new net CLED3: R14.1, U1.15 (PC3)
- no-connect marks 9 -> 11
Other:
- note added: "ATtiny816 SOIC-20"
- note added: "CLED0"
- note added: "CLED1"
- note added: "CLED2"
- note added: "CLED3"
- note removed: "ATtiny814 SOIC-14"
- moved on the sheet: D1, J1, J2, R5, R6, R7, SW1, SW2
